File: kitchen_light_controller.kicad_sch (KiCad schematic)
At the start: 15 parts, among them J1 1935161, J2 1935161, J3 1935161, J4 1935161, J5 1935161, J6 Conn_01x03, U1 SC0915, U2 VND7140AJTR

Commit message: Added readme
Connections:
- net GND: now also U1.A (USB_SHIELD), U1.B (USB_SHIELD), U1.C (USB_SHIELD), U1.D (USB_SHIELD)
Changed lines of the file:
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@@
+    )
+  )
+  (symbol (lib_id "power:GND") (at 76.2 176.53 90) (unit 1)
+    (in_bom yes) (on_board yes) (dnp no) (fields_autoplaced)
+    (property "Reference" "#PWR014" (at 82.55 176.53 0)
+      (effects (font (size 1.27 1.27)) hide)
+    )
+    (property "Value" "GND" (at 80.01 177.165 90)
+      (effects (font (size 1.27 1.27)) (justify right))
+    )
+    (property "Footprint" "" (at 76.2 176.53 0)
+      (effects (font (size 1.27 1.27)) hide)
+    )
+    (property "Datasheet" "" (at 76.2 176.53 0)
+      (effects (font (size 1.27 1.27)) hide)
+    )
+    (pin "1")
+    (instances
+      (project "kitchen_light_controller"
+        (path "/b7dbd127-2340-4bb0-b060-ce4a2230bf8a"
+          (reference "#PWR014") (unit 1)
+        )
+      )
     )
   )
